File: Microcontroller/Hernans Schematic/Senior Design.sch (KiCad schematic (older format))
At the start: 20 parts, among them IC1 BM71BLE01FC2-0B04AA, U1 MAX30102EFD+T, U2 ADXL345BCCZ-RL, U3 ATSAME70J19A-AN, U4 STBC03JR

Commit message: Add files via upload
Parts:
- removed C4: 4.7 uF, symbol Device:C
- removed D1: LED, symbol Device:LED
- removed R2, R3, R4: 10K, symbol Device:R
- removed U4: STBC03JR, BGA30N40P6X5_259X225X60N, symbol STBC03JR:STBC03JR
- added B1: 1.8-5V, Adafruit PowerBoost 500C:JSTPH2, symbol Adafruit_PowerBoost_500C-eagle-import:BATTERY
- added C1: 10uF, Adafruit PowerBoost 500C:0805-NO, symbol Adafruit_PowerBoost_500C-eagle-import:CAP_CERAMIC0805-NOOUTLINE
- added C2: 2.2uF, Adafruit PowerBoost 500C:0805-NO, symbol Adafruit_PowerBoost_500C-eagle-import:CAP_CERAMIC0805-NOOUTLINE
- added C4: 0.1uF, Adafruit PowerBoost 500C:0805-NO, symbol Adafruit_PowerBoost_500C-eagle-import:CAP_CERAMIC0805-NOOUTLINE
- added C5: 100uF/6V, Adafruit PowerBoost 500C:EIA3528-21_B-R, symbol Adafruit_PowerBoost_500C-eagle-import:CAP_TANTALUMB_3528_REFLOW
- added C6: 10µF, Adafruit PowerBoost 500C:0805-NO, symbol Adafruit_PowerBoost_500C-eagle-import:CAP_CERAMIC0805-NOOUTLINE
- added CN1: USBA_FEMALE, Adafruit PowerBoost 500C:USB_HOST-PTH, symbol Adafruit_PowerBoost_500C-eagle-import:USB_TYPEAPTHFML
- added JP1: PINHD-1X6CB, Adafruit PowerBoost 500C:1X06-CLEANBIG, symbol Adafruit_PowerBoost_500C-eagle-import:PINHD-1X6CB
- added JP2: HEADER-1X2ROUND, Adafruit PowerBoost 500C:1X02_ROUND, symbol Adafruit_PowerBoost_500C-eagle-import:HEADER-1X2ROUND
- added L1: VLC5045-6.8uH, Adafruit PowerBoost 500C:INDUCTOR_5X5MM_TDK_VLC5045, symbol Adafruit_PowerBoost_500C-eagle-import:INDUCTORTDK_VLC5045
- added LBO1: RED, Adafruit PowerBoost 500C:CHIPLED_0805_NOOUTLINE, symbol Adafruit_PowerBoost_500C-eagle-import:LED0805_NOOUTLINE
- added LED3: ORANGE, Adafruit PowerBoost 500C:CHIPLED_0805_NOOUTLINE, symbol Adafruit_PowerBoost_500C-eagle-import:LED0805_NOOUTLINE
- added LED4: GREEN, Adafruit PowerBoost 500C:CHIPLED_0805_NOOUTLINE, symbol Adafruit_PowerBoost_500C-eagle-import:LED0805_NOOUTLINE
- added PWR1: BLUE, Adafruit PowerBoost 500C:CHIPLED_0805_NOOUTLINE, symbol Adafruit_PowerBoost_500C-eagle-import:LED0805_NOOUTLINE
- added Q1: MMUN2133LT1G, Adafruit PowerBoost 500C:SC59-BEC, symbol Adafruit_PowerBoost_500C-eagle-import:-PNP_DRIVER-SC59-BEC
- added R1, R3: 1.87Mohm, Adafruit PowerBoost 500C:0805-NO, symbol Adafruit_PowerBoost_500C-eagle-import:RESISTOR0805_NOOUTLINE
- added R10, R12: 49.9K 1%, Adafruit PowerBoost 500C:0805-NO, symbol Adafruit_PowerBoost_500C-eagle-import:RESISTOR0805_NOOUTLINE
- added R11, R9: 75K 1%, Adafruit PowerBoost 500C:0805-NO, symbol Adafruit_PowerBoost_500C-eagle-import:RESISTOR0805_NOOUTLINE
- added R13, R2: 340K, Adafruit PowerBoost 500C:0805-NO, symbol Adafruit_PowerBoost_500C-eagle-import:RESISTOR0805_NOOUTLINE
- added R20, R5, R7: 1K, Adafruit PowerBoost 500C:0805-NO, symbol Adafruit_PowerBoost_500C-eagle-import:RESISTOR0805_NOOUTLINE
- added R4: 200K, Adafruit PowerBoost 500C:0805-NO, symbol Adafruit_PowerBoost_500C-eagle-import:RESISTOR0805_NOOUTLINE
- added R6: 470, Adafruit PowerBoost 500C:0805-NO, symbol Adafruit_PowerBoost_500C-eagle-import:RESISTOR0805_NOOUTLINE
- added R8: 2k, Adafruit PowerBoost 500C:0805-NO, symbol Adafruit_PowerBoost_500C-eagle-import:RESISTOR0805_NOOUTLINE
- added U1: TPS61090RSAR, Adafruit PowerBoost 500C:PVQFN-16, symbol Adafruit_PowerBoost_500C-eagle-import:VREG_TPS6103X
- added U2: MCP73831T-2ACI/OT, Adafruit PowerBoost 500C:SOT23-5, symbol Adafruit_PowerBoost_500C-eagle-import:MCP73831_2
- added X1: TERMBLOCK_1X2, Adafruit PowerBoost 500C:TERMBLOCK_1X2-3.5MM, symbol Adafruit_PowerBoost_500C-eagle-import:TERMBLOCK_1X2
- added X2: microUSB, Adafruit PowerBoost 500C:4UCONN_20329, symbol Adafruit_PowerBoost_500C-eagle-import:USBMICRO_20329
- BM71BLE01FC2-0B04AA: renamed from IC1; value BM71BLE01FC2-0B04AA -> IC?
Connections:
- net labels added: 5.0V, CSAx, ENABLE, INT1, INT2, INT3, LBO, LED0, LEDQ, PAIRING_KEY, RST_N, SCLAx, SCLSn, SDAAx, SDASn, SDOAx, STATUS1, STATUS2, SYSTEM_CONFIG, UART_CTS, UART_RTS, UART_RX_IND, UART_TX_IND, VBAT
- net labels removed: BATMS, HCI_EXD, IN, NRST, P1_7, PB2, PB3, VLED+
- wire segments 81 -> 178
- no-connect marks 62 -> 26
Other:
- note added: "2.0K = 500mA"
- note added: "6.8uH power\nw/2A current"
- note added: "Adafruit Powerboost 5000 (Battery Charger)"
- note added: "R2 < 500K\nR1 = 5.5*R2 (3.2V LBO)"
- note added: "R4 = 200K\nR3 = 1.85Mohm"
- note added: "See Pg 15\n1st para"
- note removed: "STBC03JR (Battery Charger)"
- moved on the sheet: BM71BLE01FC2-0B04AA, R1, R10, R11, R12, R13, R5, R6, R7, R8, R9, U1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
